File: esp8266-flipperzero/esp8266-flipperzero.kicad_pcb (KiCad board)
At the start: 2 copper layers, 61.3 x 28.8 mm, 11 parts, among them J1 Conn_01x08_Pin, J2 Conn_01x10_Pin, J3 USB_B_Micro, SW1 RESET button, U1 ESP-12E, U2 CH340C, U4 MCP1700x-330xxTO

Commit message: Add files via upload
Parts:
- turned U2 to 0 degrees
Routing:
- net Net-(J2-RX): track 0.00 -> 48.2 mm, vias 0 -> 3
- net Net-(SW1A-C): track 0.00 -> 46.7 mm, vias 0 -> 2
- net Net-(J2-TX): track 0.00 -> 45.8 mm, vias 0 -> 3
- net Net-(J1-A4): track 0.00 -> 37.4 mm, vias 0 -> 2
- net +3.3V: track 0.00 -> 29.2 mm, vias 0 -> 2
- net Net-(J1-B3): track 0.00 -> 24.5 mm, vias 0 -> 1
- net Net-(J1-B2): track 0.00 -> 18.1 mm, vias 0 -> 1
- net Net-(J3-VBUS): track 0.00 -> 17.2 mm, vias 0 -> 2
- net Net-(J3-D-): track 0.00 -> 14.3 mm
- net Net-(J3-D+): track 0.00 -> 12.6 mm
- net Net-(J1-C3): track 0.00 -> 12.4 mm, vias 0 -> 1
- net Net-(J2-C0): track 0.00 -> 8.04 mm
- added copper zone on F.Cu, net GND

Commit message: Add files via upload
Parts:
- moved H1 1.00 mm to (101.8, 79.0)
- moved H3 1.00 mm to (156.6, 79.0)
Routing:
- net GND: track 0.00 -> 2.57 mm
Changed lines of the file:
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@@
   )
   (footprint "MountingHole:MountingHole_3.2mm_M3" (layer "F.Cu")
-    (at 156.642 80)
+    (at 156.642 79)
     (descr "Mounting Hole 3.2mm, no annular, M3")
     (tags "mounting hole 3.2mm no annular m3")
@@
   )
   (footprint "MountingHole:MountingHole_3.2mm_M3" (layer "F.Cu")
-    (at 101.778 80)
+    (at 101.778 79)
     (descr "Mounting Hole 3.2mm, no annular, M3")
     (tags "mounting hole 3.2mm no annular m3")
@@
   (segment (start 110.16 85) (end 120.066 75.094) (width 0.25) (layer "B.Cu") (net 26))
   (segment (start 120.066 75.094) (end 124.892 75.094) (width 0.25) (layer "B.Cu") (net 26))
+  (segment (start 136.83 66.712) (end 136.068 67.474) (width 0.25) (layer "F.Cu") (net 27))
+  (segment (start 137.308 65.564) (end 137.308 66.488) (width 0.25) (layer "F.Cu") (net 27))
+  (segment (start 137.308 66.488) (end 137.084 66.712) (width 0.25) (layer "F.Cu") (net 27))
+  (segment (start 137.084 66.712) (end 136.83 66.712) (width 0.25) (layer "F.Cu") (net 27))
   (segment (start 107.62 85) (end 107.62 83.476) (width 0.25) (layer "F.Cu") (net 28))
   (segment (start 126.416 67.728) (end 126.472 67.672) (width 0.25) (layer "F.Cu") (net 28))

Commit message: Add files via upload
Parts:
- moved J3 0.14 mm to (138.6, 63.8)
Routing:
- net GND: track 2.57 -> 0.00 mm
Changed lines of the file:
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@@
   )
   (footprint "Connector_USB:USB_Micro-B_Wuerth_629105150521" (layer "F.Cu")
-    (at 138.608 63.664 180)
+    (at 138.625 63.8 180)
     (descr "USB Micro-B receptacle, http://www.mouser.com/ds/2/445/629105150521-469306.pdf")
     (tags "usb micro receptacle")
@@
   (segment (start 110.16 85) (end 120.066 75.094) (width 0.25) (layer "B.Cu") (net 26))
   (segment (start 120.066 75.094) (end 124.892 75.094) (width 0.25) (layer "B.Cu") (net 26))
-  (segment (start 136.83 66.712) (end 136.068 67.474) (width 0.25) (layer "F.Cu") (net 27))
-  (segment (start 137.308 65.564) (end 137.308 66.488) (width 0.25) (layer "F.Cu") (net 27))
-  (segment (start 137.308 66.488) (end 137.084 66.712) (width 0.25) (layer "F.Cu") (net 27))
-  (segment (start 137.084 66.712) (end 136.83 66.712) (width 0.25) (layer "F.Cu") (net 27))
   (segment (start 107.62 85) (end 107.62 83.476) (width 0.25) (layer "F.Cu") (net 28))
   (segment (start 126.416 67.728) (end 126.472 67.672) (width 0.25) (layer "F.Cu") (net 28))
@@
     (polygon
       (pts
-        (xy 160.198 59.092)
-        (xy 160.452 89.826)
-        (xy 113.716 89.318)
-        (xy 113.716 58.076)
+        (xy 161 58)
+        (xy 161 89.826)
+        (xy 114 90)
+        (xy 114 58)
       )
     )
