File: esp8266-flipperzero/esp8266-flipperzero.kicad_sch (KiCad schematic)
At the start: 11 parts, among them J1 Conn_01x08_Pin, J2 Conn_01x10_Pin, J3 USB_B_Micro, SW1 RESET button, U1 ESP-12E, U2 CH340C, U4 MCP1700x-330xxTO

Commit message: Add files via upload
Parts:
- H1, H2, H3, H4: footprint (none) -> MountingHole:MountingHole_3.2mm_M3
Changed lines of the file:
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@@
       (effects (font (size 1.27 1.27)) (justify left))
     )
-    (property "Footprint" "" (at 262.89 29.845 0)
+    (property "Footprint" "MountingHole:MountingHole_3.2mm_M3" (at 262.89 29.845 0)
       (effects (font (size 1.27 1.27)) hide)
     )
@@
       (effects (font (size 1.27 1.27)) (justify left))
     )
-    (property "Footprint" "" (at 262.89 35.56 0)
+    (property "Footprint" "MountingHole:MountingHole_3.2mm_M3" (at 262.89 35.56 0)
       (effects (font (size 1.27 1.27)) hide)
     )
@@
       (effects (font (size 1.27 1.27)) (justify left))
     )
-    (property "Footprint" "" (at 262.89 46.99 0)
+    (property "Footprint" "MountingHole:MountingHole_3.2mm_M3" (at 262.89 46.99 0)
       (effects (font (size 1.27 1.27)) hide)
     )
@@
       (effects (font (size 1.27 1.27)) (justify left))
     )
-    (property "Footprint" "" (at 262.89 41.275 0)
-      (effects (font (size 1.27 1.27)) hide)
-    )
+    (property "Footprint" "MountingHole:MountingHole_3.2mm_M3" (at 262.89 41.275 0)
+      (effects (font (size 1.27 1.27)) hide)
+    )
